File: amplification.kicad_sch (KiCad schematic)
At the start: 34 parts, among them Q1 PNP, Q10 PNP, Q11 NPN, Q12 NPN, Q13 NPN, Q14 PNP, Q15 NPN, Q16 PNP, Q2 PNP, Q3 NPN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

Commit message: organize amp sheet
Connections:
- net +24V: no longer Q13.1 (C), Q15.1 (C), Q2.3 (E), R9.1
- new net: Q13.1 (C), Q15.1 (C), Q2.3 (E), R9.1
Other:
- moved on the sheet: Q10, Q11, Q7, Q8, Q9, R14, R15, R16, R17

Commit message: initial component placement in pcb
Parts:
- removed R22, R23: R, Resistor_SMD:R_0603_1608Metric, symbol Device:R
- added C3: C, symbol Device:C
- added Q17: NPN, D44H8:TO-220_STM, symbol Simulation_SPICE:NPN
- added Q18: PNP, D44H8:TO-220_STM, symbol Simulation_SPICE:PNP
- Q1, Q10, Q11, Q12, Q13, Q14, Q2, Q3, Q4, Q5, Q6, Q7, Q8, Q9: footprint (none) -> 2N5401:P210_TO-92
- Q15, Q16: footprint (none) -> D44H8:TO-220_STM
- R10, R11, R12, R13, R14, R15, R16, R17, R18, R19, R20, R21, R6, R7, R8, R9: footprint Resistor_SMD:R_0603_1608Metric -> Resistor_THT:R_Axial_DIN0207_L6.3mm_D2.5mm_P7.62mm_Horizontal
Connections:
- net +24V: now also Q13.1 (C), Q15.1 (C), Q2.3 (E), R9.1, Q17.1 (C)
- net -24V: now also Q18.1 (C)
- net amp_out: now also Q15.3 (E), Q16.3 (E), Q17.3 (E), Q18.3 (E)
- net at Q14.3 (E), Q16.2 (B), R21.2: now also Q18.2 (B)
- net at Q13.3 (E), Q15.2 (B), R20.1: now also Q17.2 (B)
- net at Q1.1 (C), Q3.1 (C), Q7.1 (C)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: now also C3.2
- net at Q11.1 (C), Q12.3 (E), Q14.2 (B)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: now also C3.1
Other:
- moved on the sheet: Q1, Q10, Q11, Q12, Q13, Q14, Q15, Q16, Q2, Q3, Q4, Q5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

Commit message: RAAAAH Let's gooo to production baby
Parts:
- C3: footprint (none) -> Capacitor_THT:C_Disc_D5.0mm_W2.5mm_P5.00mm
Changed lines of the file:
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@@
 	(label "amp_out_fb"
 		(at 130.81 91.44 180)
-		(fields_autoplaced yes)
 		(effects
 			(font
@@
 	(label "amp_out_fb"
 		(at 254 95.25 0)
-		(fields_autoplaced yes)
 		(effects
 			(font
@@
 		(shape input)
 		(at 34.29 97.79 180)
-		(fields_autoplaced yes)
 		(effects
 			(font
@@
 		(shape output)
 		(at 266.7 95.25 0)
-		(fields_autoplaced yes)
 		(effects
 			(font
@@
 			)
 		)
-		(property "Footprint" ""
+		(property "Footprint" "Capacitor_THT:C_Disc_D5.0mm_W2.5mm_P5.00mm"
 			(at 138.1252 127 0)
 			(effects
