File: baxandall.kicad_sch (KiCad schematic)
At the start: 10 parts, among them U1 NE5532

Commit message: initial component placement in pcb
Parts:
- R1, R2, R3, R4, R5: footprint Resistor_SMD:R_0603_1608Metric -> Resistor_THT:R_Axial_DIN0207_L6.3mm_D2.5mm_P7.62mm_Horizontal
- U1: footprint NE5532DR:D8 -> NE5532DR:D8-M
Changed lines of the file:
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@@
 			)
 		)
-		(property "Footprint" "Resistor_SMD:R_0603_1608Metric"
+		(property "Footprint" "Resistor_THT:R_Axial_DIN0207_L6.3mm_D2.5mm_P7.62mm_Horizontal"
 			(at 85.09 53.848 90)
 			(effects
@@
 			)
 		)
-		(property "Footprint" "NE5532DR:D8"
+		(property "Footprint" "NE5532DR:D8-M"
 			(at 118.11 66.04 0)
 			(effects
@@
 			)
 		)
-		(property "Footprint" "Resistor_SMD:R_0603_1608Metric"
+		(property "Footprint" "Resistor_THT:R_Axial_DIN0207_L6.3mm_D2.5mm_P7.62mm_Horizontal"
 			(at 93.472 59.69 90)
 			(effects
@@
 			)
 		)
-		(property "Footprint" "Resistor_SMD:R_0603_1608Metric"
+		(property "Footprint" "Resistor_THT:R_Axial_DIN0207_L6.3mm_D2.5mm_P7.62mm_Horizontal"
 			(at 105.41 53.848 90)
 			(effects
@@
 			)
 		)
-		(property "Footprint" "Resistor_SMD:R_0603_1608Metric"
+		(property "Footprint" "Resistor_THT:R_Axial_DIN0207_L6.3mm_D2.5mm_P7.62mm_Horizontal"
 			(at 105.41 79.248 90)
 			(effects
@@
 			)
 		)
-		(property "Footprint" "Resistor_SMD:R_0603_1608Metric"
+		(property "Footprint" "Resistor_THT:R_Axial_DIN0207_L6.3mm_D2.5mm_P7.62mm_Horizontal"
 			(at 85.09 79.248 90)
 			(effects

Commit message: feat: updated schematic
Parts:
- RV4, RV5: footprint (none) -> Potentiometer_THT:Potentiometer_Alps_RK163_Single_Horizontal
Changed lines of the file:
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@@
 		(shape input)
 		(at 63.5 66.04 180)
+		(fields_autoplaced yes)
 		(effects
 			(font
@@
 		(shape output)
 		(at 140.97 66.04 0)
+		(fields_autoplaced yes)
 		(effects
 			(font
@@
 			)
 		)
-		(property "Footprint" ""
+		(property "Footprint" "Potentiometer_THT:Potentiometer_Alps_RK163_Single_Horizontal"
 			(at 95.25 52.07 0)
 			(effects
@@
 			)
 		)
-		(property "Footprint" ""
+		(property "Footprint" "Potentiometer_THT:Potentiometer_Alps_RK163_Single_Horizontal"
 			(at 95.25 77.47 0)
 			(effects

Commit message: RAAAAH Let's gooo to production baby
Parts:
- C1, C2: footprint Capacitor_SMD:C_0603_1608Metric -> Capacitor_THT:C_Disc_D5.0mm_W2.5mm_P5.00mm
- U1: footprint NE5532DR:D8-M -> Package_DIP:DIP-8_W7.62mm_Socket
Changed lines of the file:
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@@
 		(shape input)
 		(at 63.5 66.04 180)
-		(fields_autoplaced yes)
 		(effects
 			(font
@@
 		(shape output)
 		(at 140.97 66.04 0)
-		(fields_autoplaced yes)
 		(effects
 			(font
@@
 			)
 		)
-		(property "Footprint" "Capacitor_SMD:C_0603_1608Metric"
+		(property "Footprint" "Capacitor_THT:C_Disc_D5.0mm_W2.5mm_P5.00mm"
 			(at 94.2848 66.04 0)
 			(effects
@@
 			)
 		)
-		(property "Footprint" "NE5532DR:D8-M"
+		(property "Footprint" "Package_DIP:DIP-8_W7.62mm_Socket"
 			(at 118.11 66.04 0)
 			(effects
@@
 			)
 		)
-		(property "Footprint" "Capacitor_SMD:C_0603_1608Metric"
+		(property "Footprint" "Capacitor_THT:C_Disc_D5.0mm_W2.5mm_P5.00mm"
 			(at 99.06 40.9448 0)
 			(effects
